File: rev_c/dual_slot_encoders.sch (KiCad schematic (older format))
At the start: 15 parts, among them U1 GP1S094HCZ0F, U2 GP1S094HCZ0F, U3 GPS1S97HCZ0F, U4 GPS1S97HCZ0F

Commit message: Rev. C is pretty much done.
Parts:
- removed N1: ENCODER_CONNECTOR, symbol ENCODER_CONNECTOR
- added N1: MOTOR_ENCODER_CONN, dual_slot_encoders:Pin_Header_Straight_2x04_Shrouded, symbol MOTOR_ENCODER_CONN
- added N2: MOTOR_CONN, dual_slot_encoders:5MM_TERMINAL_BLOCK_2_POS, symbol MOTOR_CONN
- G1: renamed from Z1; footprint (none) -> dual_slot_encoders:OSHW_LOGO_200mil
- H1, H2, H3, H4: footprint (none) -> dual_slot_encoders:MountingHole_3mm
- R1, R2, R3, R4: footprint (none) -> dual_slot_encoders:Resistor_Horizontal_400
- TP1: footprint (none) -> dual_slot_encoders:Pin_Header_Straight_1x01
- U1, U2: footprint (none) -> dual_slot_encoders:GP1S094HCZ0F
- U3, U4: footprint (none) -> dual_slot_encoders:GP1S097HCZ0F
Connections:
- net 5V: now also N1.8 (VCC)
- net A: now also N1.1 (QUAD_A)
- net B: now also N1.7 (QUAD_B)
- net GND: now also N1.2 (LGND)
- new net MOTOR+: N1.5 (MOTOR_B), N1.6 (MOTOR_B), N2.2 (+)
- new net MOTOR-: N1.3 (MOTOR_A), N1.4 (MOTOR_A), N2.1 (-)
Other:
- moved on the sheet: R1
Changed lines of the file:
@@
 Sheet 1 1
 Title "Quadrature Dual Slot Encoders"
-Date "29 Jul 2014"
-Rev "B"
+Date "Sun 05 Oct 2014"
+Rev "C"
 Comp ""
 Comment1 ""
@@
 F 0 "R2" H 3670 1950 50  0000 L CNN
 F 1 "10K" H 3670 1850 50  0000 L CNN
-F 2 "" H 3600 1950 60  0000 C CNN
+F 2 "dual_slot_encoders:Resistor_Horizontal_400" H 3600 1950 60  0001 C CNN
 F 3 "" H 3600 1950 60  0000 C CNN
 	1    3600 1900
@@
 F 0 "H1" H 4050 4950 50  0000 C CNN
 F 1 "3MM_HOLE" H 4100 4650 50  0000 C CNN
-F 2 "" H 4100 4800 60  0000 C CNN
+F 2 "dual_slot_encoders:MountingHole_3mm" H 4100 4800 60  0001 C CNN
 F 3 "" H 4100 4800 60  0000 C CNN
 	1    4100 4800
@@
 F 0 "U3" H 6550 3195 50  0000 C CNN
 F 1 "GPS1S97HCZ0F" H 6850 2445 50  0000 C CNN
-F 2 "" H 7200 2700 60  0000 C CNN
+F 2 "dual_slot_encoders:GP1S097HCZ0F" H 7200 2700 60  0001 C CNN
 F 3 "" H 7200 2700 60  0000 C CNN
 	1    6850 2900
@@
 F 0 "U4" H 6550 4095 50  0000 C CNN
 F 1 "GPS1S97HCZ0F" H 6850 3345 50  0000 C CNN
-F 2 "" H 7200 3600 60  0000 C CNN
+F 2 "dual_slot_encoders:GP1S097HCZ0F" H 7200 3600 60  0001 C CNN
 F 3 "" H 7200 3600 60  0000 C CNN
 	1    6850 3800
@@
 F 0 "U1" H 4150 3195 50  0000 C CNN
 F 1 "GP1S094HCZ0F" H 4450 2445 50  0000 C CNN
-F 2 "" H 4800 2700 60  0000 C CNN
+F 2 "dual_slot_encoders:GP1S094HCZ0F" H 4800 2700 60  0001 C CNN
 F 3 "" H 4800 2700 60  0000 C CNN
 	1    4450 2900
@@
 F 0 "U2" H 4150 4095 50  0000 C CNN
 F 1 "GP1S094HCZ0F" H 4450 3345 50  0000 C CNN
-F 2 "" H 4800 3600 60  0000 C CNN
+F 2 "dual_slot_encoders:GP1S094HCZ0F" H 4800 3600 60  0001 C CNN
 F 3 "" H 4800 3600 60  0000 C CNN
 	1    4450 3800
@@
 F 0 "R3" H 5370 1900 50  0000 L CNN
 F 1 "470" H 5370 1800 50  0000 L CNN
-F 2 "" H 5300 1900 60  0000 C CNN
+F 2 "dual_slot_encoders:Resistor_Horizontal_400" H 5300 1900 60  0001 C CNN
 F 3 "" H 5300 1900 60  0000 C CNN
 	1    5300 1850
@@
 L R_VERT R1
 U 1 1 53C161E7
-P 3100 1900
-F 0 "R1" H 3170 1950 50  0000 L CNN
-F 1 "10K" H 3170 1850 50  0000 L CNN
-F 2 "" H 3100 1950 60  0000 C CNN
-F 3 "" H 3100 1950 60  0000 C CNN
-	1    3100 1900
-	1    0    0    -1
-$EndComp
-Wire Wire Line
-	3100 2100 3100 3600
+P 3100 2100
+F 0 "R1" H 3170 2150 50  0000 L CNN
+F 1 "10K" H 3170 2050 50  0000 L CNN
+F 2 "dual_slot_encoders:Resistor_Horizontal_400" H 3100 2150 60  0001 C CNN
+F 3 "" H 3100 2150 60  0000 C CNN
+	1    3100 2100
+	1    0    0    -1
+$EndComp
+Wire Wire Line
+	3100 2300 3100 3600
 Wire Wire Line
 	7700 2200 5300 2200
@@
 F 0 "H2" H 4050 5350 50  0000 C CNN
 F 1 "3MM_HOLE" H 4100 5050 50  0000 C CNN
-F 2 "" H 4100 5200 60  0000 C CNN
+F 2 "dual_slot_encoders:MountingHole_3mm" H 4100 5200 60  0001 C CNN
 F 3 "" H 4100 5200 60  0000 C CNN
 	1    4100 5200
@@
 F 0 "H3" H 4050 5750 50  0000 C CNN
 F 1 "3MM_HOLE" H 4100 5450 50  0000 C CNN
-F 2 "" H 4100 5600 60  0000 C CNN
+F 2 "dual_slot_encoders:MountingHole_3mm" H 4100 5600 60  0001 C CNN
 F 3 "" H 4100 5600 60  0000 C CNN
 	1    4100 5600
@@
 F 0 "H4" H 4050 6150 50  0000 C CNN
 F 1 "3MM_HOLE" H 4100 5850 50  0000 C CNN
-F 2 "" H 4100 6000 60  0000 C CNN
+F 2 "dual_slot_encoders:MountingHole_3mm" H 4100 6000 60  0001 C CNN
 F 3 "" H 4100 6000 60  0000 C CNN
 	1    4100 6000
@@
 	3800 5600 3700 5600
 Connection ~ 3700 5600
-$Comp
-L ENCODER_CONNECTOR N1
-U 1 1 53C169C0
-P 2300 1550
-F 0 "N1" H 2300 1800 50  0000 C CNN
-F 1 "ENCODER_CONNECTOR" H 2300 1300 50  0000 C CNN
-F 2 "" H 2300 1550 60  0000 C CNN
-F 3 "" H 2300 1550 60  0000 C CNN
-	1    2300 1550
-	-1   0    0    -1
-$EndComp
 Wire Wire Line
 	2900 4500 2900 1700
 Wire Wire Line
-	2900 1700 2600 1700
-Wire Wire Line
-	3100 1700 3100 1600
-Wire Wire Line
-	3100 1600 2600 1600
-Wire Wire Line
-	3600 1700 3600 1500
-Wire Wire Line
-	3600 1500 2600 1500
-Wire Wire Line
-	5300 1650 5300 1400
-Wire Wire Line
-	2600 1400 7800 1400
+	2900 1700 2200 1700
+Wire Wire Line
+	3100 1900 3100 1800
+Wire Wire Line
+	3100 1800 2200 1800
+Wire Wire Line
+	3600 1700 3600 1200
+Wire Wire Line
+	3600 1200 2200 1200
+Wire Wire Line
+	5300 1650 5300 1100
+Wire Wire Line
+	2200 1100 7800 1100
 Text Notes 4150 4450 0    50   ~ 0
 3mm Slot Gap\n.3mm Slit Width
-Text Label 2700 1700 0    50   ~ 0
+Text Label 2400 1700 0    50   ~ 0
 GND
-Text Label 2700 1400 0    50   ~ 0
+Text Label 2400 1100 0    50   ~ 0
 5V
-Text Label 2700 1600 0    50   ~ 0
+Text Label 2400 1800 0    50   ~ 0
 A
-Text Label 2700 1500 0    50   ~ 0
+Text Label 2400 1200 0    50   ~ 0
 B
 $Comp
-L OSHW_LOGO Z1
+L OSHW_LOGO G1
 U 1 1 53C1B3B3
 P 5000 5250
-F 0 "Z1" H 5000 5400 50  0000 C CNN
+F 0 "G1" H 5000 5400 50  0000 C CNN
 F 1 "OSHW_LOGO" H 5000 5100 50  0000 C CNN
-F 2 "" H 5000 5250 50  0000 C CNN
+F 2 "dual_slot_encoders:OSHW_LOGO_200mil" H 5000 5250 50  0001 C CNN
 F 3 "" H 5000 5250 50  0000 C CNN
 	1    5000 5250
@@
 F 0 "R4" H 7870 1900 50  0000 L CNN
 F 1 "470" H 7870 1800 50  0000 L CNN
-F 2 "" H 7800 1900 60  0000 C CNN
+F 2 "dual_slot_encoders:Resistor_Horizontal_400" H 7800 1900 60  0001 C CNN
 F 3 "" H 7800 1900 60  0000 C CNN
 	1    7800 1850
@@
 	7700 2700 7700 2200
 Wire Wire Line
-	7800 1400 7800 1650
-Connection ~ 5300 1400
+	7800 1100 7800 1650
+Connection ~ 5300 1100
 Wire Wire Line
 	7800 2050 7800 3600
@@
 F 0 "TP1" H 8100 4650 50  0000 C CNN
 F 1 "GND" H 8100 4350 50  0000 C CNN
-F 2 "" H 8100 4500 60  0000 C CNN
+F 2 "dual_slot_encoders:Pin_Header_Straight_1x01" H 8100 4500 60  0001 C CNN
 F 3 "" H 8100 4500 60  0000 C CNN
 	1    8100 4500
@@
 Text Notes 4550 4950 0    60   ~ 0
 Note:\n  Only install one pair of slot interrutpers.\n  Either install U1/U2 or U3/U4.\n  Do not install both pairs.
+$Comp
+L MOTOR_ENCODER_CONN N1
+U 1 1 5431825B
+P 1800 1450
+F 0 "N1" H 1800 1900 50  0000 C CNN
+F 1 "MOTOR_ENCODER_CONN" H 1800 1000 50  0000 C CNN
+F 2 "dual_slot_encoders:Pin_Header_Straight_2x04_Shrouded" H 1800 1450 60  0001 C CNN
+F 3 "" H 1800 1450 60  0000 C CNN
+	1    1800 1450
+	-1   0    0    1
+$EndComp
+Wire Wire Line
+	2200 1400 3000 1400
+Wire Wire Line
+	2300 1400 2300 1300
+Wire Wire Line
+	2300 1300 2200 1300
+Wire Wire Line
+	2200 1600 2300 1600
+Wire Wire Line
+	2300 1600 2300 1500
+Wire Wire Line
+	2200 1500 3000 1500
+$Comp
+L MOTOR_CONN N2
+U 1 1 543185E5
+P 3300 1450
+F 0 "N2" H 3300 1600 50  0000 C CNN
+F 1 "MOTOR_CONN" H 3300 1300 50  0000 C CNN
+F 2 "dual_slot_encoders:5MM_TERMINAL_BLOCK_2_POS" H 3300 1450 60  0001 C CNN
+F 3 "" H 3300 1450 60  0000 C CNN
+	1    3300 1450
+	1    0    0    -1
+$EndComp
+Connection ~ 2300 1400
+Connection ~ 2300 1500
+Text Label 2400 1400 0    50   ~ 0
+MOTOR+
+Text Label 2400 1500 0    50   ~ 0
+MOTOR-
 $EndSCHEMATC
