File: rev_e/dual_slot_encoders.sch (KiCad schematic (older format))
At the start: 14 parts, among them U1 GP1S094HCZ0F, U2 GP1S094HCZ0F, U3 GPS1S97HCZ0F, U4 GPS1S97HCZ0F

Commit message: Got Rev. E wrapped up.
Parts:
- N1: footprint ~ -> (none)
Connections:
- net A: now also N1.5 (QUAD_A); no longer N1.4 (LGND)
- net B: now also N1.6 (QUAD_B); no longer N1.7 (LED_EN)
- net LED_EN: now also N1.7 (LED_EN); no longer N1.6 (QUAD_B)
- net LGND: now also N1.4 (LGND); no longer N1.5 (QUAD_A)
Changed lines of the file:
@@
 LIBS:valves
 LIBS:dual_slot_encoders-cache
-EELAYER 24 0
+EELAYER 25 0
 EELAYER END
 $Descr A 11000 8500
@@
 Sheet 1 1
 Title "Quadrature Dual Slot Encoders"
-Date "Sat 11 Oct 2014"
-Rev "D"
+Date "Thu 30 Oct 2014"
+Rev "E"
 Comp ""
 Comment1 ""
@@
 Text Notes 3750 5950 0    50   ~ 0
 3mm Slot Gap\n.3mm Slit Width
-Text Label 2100 2100 0    50   ~ 0
+Text Label 2100 2200 0    50   ~ 0
 LED_EN
 Text Label 2100 1800 0    50   ~ 0
 LPWR
-Text Label 2100 1900 0    50   ~ 0
+Text Label 2100 2000 0    50   ~ 0
 A
-Text Label 2100 2200 0    50   ~ 0
+Text Label 2100 2100 0    50   ~ 0
 B
 $Comp
@@
 F 0 "N1" H 1400 2600 50  0000 C CNN
 F 1 "MOTOR_ENCODER_CONN_2X5" H 1400 1500 50  0000 C CNN
-F 2 "~" H 1200 1000 60  0000 C CNN
+F 2 "" H 1400 2050 60  0000 C CNN
 F 3 "" H 1400 2050 60  0000 C CNN
 	1    1400 2050
 	-1   0    0    -1
 $EndComp
-Text Label 2100 2000 0    50   ~ 0
+Text Label 2100 1900 0    50   ~ 0
 LGND
 Text Label 2100 2300 0    50   ~ 0
@@
 	4800 4500 6800 4500
 Wire Wire Line
-	6800 4500 6800 2200
+	6800 4500 6800 2100
 Wire Wire Line
 	3400 5500 2900 5500
@@
 	4800 6100 7000 6100
 Wire Wire Line
-	7000 6100 7000 1900
+	7000 6100 7000 2000
 Connection ~ 3300 3400
 Connection ~ 2900 4900
@@
 	2900 2300 2900 2800
 Wire Wire Line
-	7000 1900 1800 1900
-Wire Wire Line
-	6800 2200 1800 2200
-Wire Wire Line
-	1800 2100 2700 2100
-Wire Wire Line
-	2700 2100 2700 6000
+	7000 2000 1800 2000
+Wire Wire Line
+	6800 2100 1800 2100
+Wire Wire Line
+	1800 2200 2700 2200
+Wire Wire Line
+	2700 2200 2700 6000
 Connection ~ 2900 6000
 Connection ~ 2900 2300
@@
 Connection ~ 4900 4800
 Wire Wire Line
-	7400 2000 1800 2000
+	7400 1900 1800 1900
 Connection ~ 4900 1800
 Wire Wire Line
@@
 Connection ~ 7000 5500
 Wire Wire Line
-	7400 2000 7400 4800
+	7400 1900 7400 4800
 Wire Wire Line
 	1900 1700 1800 1700
